File: MP3PlayerPCB/MP3PlayerPCB.kicad_sch (KiCad schematic)
At the start: 1 part, among them U1 ESP32-WROOM-32

Commit message: Save current PCB work: ESP32-CAM schematic, project settings, pin edits
Snapshot of the KiCad schematic (restored from local history) and the
uncommitted firmware pin edits before starting PCB v2. Ignore KiCad
lock files, local history and restore backups.
Parts:
- removed U1: ESP32-WROOM-32, RF_Module:ESP32-WROOM-32, symbol RF_Module:ESP32-WROOM-32
- added BT1: Battery, Connector_PinSocket_2.00mm:PinSocket_1x02_P2.00mm_Horizontal, symbol Device:Battery
- added C1, C2: 10uF, Capacitor_SMD:C_1206_3216Metric_Pad1.33x1.80mm_HandSolder, symbol Device:C_Small
- added D1: RED, LED_SMD:LED_0805_2012Metric_Pad1.15x1.40mm_HandSolder, symbol Device:LED
- added D2: GREEN, LED_SMD:LED_0805_2012Metric_Pad1.15x1.40mm_HandSolder, symbol Device:LED
- added J1: GC9A01, GC9A01:GC9A01 TFT, symbol Connector:Conn_01x07_Socket
- added J2: USB-C Connector, Connector_PinSocket_2.00mm:PinSocket_1x02_P2.00mm_Horizontal, symbol Connector:Conn_01x02_Socket
- added J3: Battery Connector, Connector_JST:JST_PH_B2B-PH-K_1x02_P2.00mm_Vertical, symbol Connector:Conn_01x02_Socket
- added R1: 3Ohms, Resistor_SMD:R_0805_2012Metric_Pad1.20x1.40mm_HandSolder, symbol Device:R
- added R2, R3: 1k, Resistor_SMD:R_0805_2012Metric_Pad1.20x1.40mm_HandSolder, symbol Device:R
- added SW1: Next, Button_Switch_THT:SW_PUSH_6mm, symbol Switch:SW_Push
- added SW2: Prev, Button_Switch_THT:SW_PUSH_6mm, symbol Switch:SW_Push
- added SW3: RotaryEncoder_Switch, Rotary_Encoder:RotaryEncoder_Alps_EC11E-Switch_Vertical_H20mm, symbol Device:RotaryEncoder_Switch
- added U1: ESP32-CAM, ESP32-CAM:ESP32-CAM, symbol ESP32-CAM:ESP32-CAM
- added U2: AP2112K-3.3, Package_TO_SOT_SMD:SOT-23-5, symbol Regulator_Linear:AP2112K-3.3
- added U3: TP4056-42-ESOP8, Package_SO:SOIC-8-1EP_3.9x4.9mm_P1.27mm_EP2.41x3.3mm_ThermalVias, symbol Battery_Management:TP4056-42-ESOP8
Connections:
- new net: R1.1, U3.2 (PROG)
- new net: R3.1, U3.6 (~{STDBY})
- new net: R2.1, U3.7 (~{CHRG})
- new net: D2.1 (K), R3.2
- new net: D1.1 (K), R2.2
- new net +3V3: J1.1 (VCC), U1.P$8 (3V3), U2.5 (VOUT)
- new net +BATT: BT1.1 (+), C1.1, J3.1 (Pin_1), U2.1 (VIN), U2.3 (EN), U3.5 (BAT)
- new net -BATT: BT1.2 (-), C1.2, C2.2, J1.2 (GND), J2.2 (Pin_2), J3.2 (Pin_2), R1.2, SW1.1, SW2.1, SW3.C, SW3.S2, U1.P$10 (GND@3), U1.P$5 (GND@2), U2.2 (GND), U3.1 (TEMP), U3.3 (GND)
- new net B1: SW2.2, U1.P$16 (GPIO4)
- new net B2: SW1.2, U1.P$2 (GPIO1)
- new net B3: SW3.S1
- new net CS: J1.6 (CS), U1.P$12 (GPIO13)
- new net DC: J1.5 (DC), U1.P$13 (GPIO15)
- new net RST: J1.7 (RST), U1.P$11 (GPIO12)
- new net RotA: SW3.A, U1.P$3 (GPIO3)
- new net RotB: SW3.B, U1.P$7 (GPIO16)
- new net SCL: J1.3 (SCL), U1.P$15 (GPIO2)
- new net SDA: J1.4 (SDA), U1.P$14 (GPIO14)
- new net VBUS: C2.1, D1.2 (A), D2.2 (A), J2.1 (Pin_1), U3.4 (V_{CC}), U3.8 (CE)
